Commit message: feat(hexapod): prepare project for Gazebo simulation (URDF physics and controllers config)

File: projects/hexapod_master/urdf/hexapod.urdf (robot description, URDF)
Before this commit: robot hexapod_master, 19 links, 18 joints
Links:
- link base_link: mass None -> 1.0; geometry collision box size=0.24 0.16 0.03; visual box size=0.24 0.16 0.03
