Commit message: feat(hexapod): add contact sensors and contact bridge for autonomous terrain feedback

File: projects/hexapod_master/urdf/hexapod.urdf.xacro (robot description, xacro)
@@ -71,4 +71,5 @@
       <xacro:box_inertia m="0.05" x="0.03" y="0.02" z="0.02"/>
     </link>
+    <gazebo reference="${prefix}_coxa_link"><material>Gazebo/Green</material></gazebo>
     <!-- Femur -->
     <joint name="${prefix}_femur_joint" type="revolute">
@@ -82,4 +83,5 @@
       <xacro:box_inertia m="0.1" x="0.05" y="0.015" z="0.015"/>
     </link>
+    <gazebo reference="${prefix}_femur_link"><material>Gazebo/DarkGrey</material></gazebo>
     <!-- Tibia -->
     <joint name="${prefix}_tibia_joint" type="revolute">
@@ -93,4 +95,25 @@
       <xacro:box_inertia m="0.1" x="0.08" y="0.01" z="0.01"/>
     </link>
+    <gazebo reference="${prefix}_tibia_link">
+      <material>Gazebo/Green</material>
+      <mu1>1.0</mu1>
+      <mu2>1.0</mu2>
+      <kp>1000000.0</kp>
+      <kd>1.0</kd>
+      <!-- Contact Sensor for Terrain Feedback -->
+      <sensor name="${prefix}_contact_sensor" type="contact">
+        <always_on>true</always_on>
+        <update_rate>50</update_rate>
+        <contact>
+          <collision>${prefix}_tibia_link_collision</collision>
+        </contact>
+        <plugin name="${prefix}_contact_plugin" filename="libgazebo_ros_contact.so">
+          <ros>
+            <namespace>/</namespace>
+            <remapping>~/out:=${prefix}_contact</remapping>
+          </ros>
+        </plugin>
+      </sensor>
+    </gazebo>
   </xacro:macro>
   <!-- Instantiate 6 Legs -->

Commit message: Hexapod: Synchronize geometry config between YAML, URDF and Python. Add reachability error handling.

File: projects/hexapod_master/urdf/hexapod.urdf.xacro (robot description, xacro)
@@ -4,4 +4,8 @@
   <xacro:property name="body_m" value="1.0" />
   <xacro:property name="leg_m" value="0.1" />
+  <!-- Leg Dimensions (Sync with hexapod_config.yaml) -->
+  <xacro:property name="l1" value="0.03" />
+  <xacro:property name="l2" value="0.05" />
+  <xacro:property name="l3" value="0.08" />
   <!-- Materials -->
   <material name="dark_gray"><color rgba="0.2 0.2 0.2 1.0"/></material>
@@ -67,7 +71,7 @@
     </joint>
     <link name="${prefix}_coxa_link">
-      <visual><origin xyz="0.015 0 0"/><geometry><box size="0.03 0.02 0.02"/></geometry><material name="green"/></visual>
-      <collision><origin xyz="0.015 0 0"/><geometry><box size="0.03 0.02 0.02"/></geometry></collision>
-      <xacro:box_inertia m="0.05" x="0.03" y="0.02" z="0.02"/>
+      <visual><origin xyz="${l1/2} 0 0"/><geometry><box size="${l1} 0.02 0.02"/></geometry><material name="green"/></visual>
+      <collision><origin xyz="${l1/2} 0 0"/><geometry><box size="${l1} 0.02 0.02"/></geometry></collision>
+      <xacro:box_inertia m="0.05" x="${l1}" y="0.02" z="0.02"/>
     </link>
     <gazebo reference="${prefix}_coxa_link"><material>Gazebo/Green</material></gazebo>
@@ -75,11 +79,11 @@
     <joint name="${prefix}_femur_joint" type="revolute">
       <parent link="${prefix}_coxa_link"/><child link="${prefix}_femur_link"/>
-      <origin xyz="0.03 0 0" rpy="0 0 0"/><axis xyz="0 1 0"/>
+      <origin xyz="${l1} 0 0" rpy="0 0 0"/><axis xyz="0 1 0"/>
       <limit lower="-1.57" upper="1.57" effort="10" velocity="1.0"/>
     </joint>
     <link name="${prefix}_femur_link">
-      <visual><origin xyz="0.025 0 0"/><geometry><box size="0.05 0.015 0.015"/></geometry><material name="dark_gray"/></visual>
-      <collision><origin xyz="0.025 0 0"/><geometry><box size="0.05 0.015 0.015"/></geometry></collision>
-      <xacro:box_inertia m="0.1" x="0.05" y="0.015" z="0.015"/>
+      <visual><origin xyz="${l2/2} 0 0"/><geometry><box size="${l2} 0.015 0.015"/></geometry><material name="dark_gray"/></visual>
+      <collision><origin xyz="${l2/2} 0 0"/><geometry><box size="${l2} 0.015 0.015"/></geometry></collision>
+      <xacro:box_inertia m="0.1" x="${l2}" y="0.015" z="0.015"/>
     </link>
     <gazebo reference="${prefix}_femur_link"><material>Gazebo/DarkGrey</material></gazebo>
@@ -87,11 +91,11 @@
     <joint name="${prefix}_tibia_joint" type="revolute">
       <parent link="${prefix}_femur_link"/><child link="${prefix}_tibia_link"/>
-      <origin xyz="0.05 0 0" rpy="0 0 0"/><axis xyz="0 1 0"/>
+      <origin xyz="${l2} 0 0" rpy="0 0 0"/><axis xyz="0 1 0"/>
       <limit lower="-3.14" upper="0" effort="10" velocity="1.0"/>
     </joint>
     <link name="${prefix}_tibia_link">
-      <visual><origin xyz="0.04 0 0"/><geometry><box size="0.08 0.01 0.01"/></geometry><material name="green"/></visual>
-      <collision><origin xyz="0.04 0 0"/><geometry><box size="0.08 0.01 0.01"/></geometry></collision>
-      <xacro:box_inertia m="0.1" x="0.08" y="0.01" z="0.01"/>
+      <visual><origin xyz="${l3/2} 0 0"/><geometry><box size="${l3} 0.01 0.01"/></geometry><material name="green"/></visual>
+      <collision><origin xyz="${l3/2} 0 0"/><geometry><box size="${l3} 0.01 0.01"/></geometry></collision>
+      <xacro:box_inertia m="0.1" x="${l3}" y="0.01" z="0.01"/>
     </link>
     <gazebo reference="${prefix}_tibia_link">

Commit message: Hexapod: Implement Stage 5 base - Add 3-DOF manipulator to URDF and Python IK logic

File: projects/hexapod_master/urdf/hexapod.urdf.xacro (robot description, xacro)
@@ -128,3 +128,39 @@
   <xacro:leg prefix="lm" x="0.0"   y="0.10"  yaw="1.571"/>
   <xacro:leg prefix="lb" x="-0.12" y="0.08"  yaw="2.356"/>
+  <!-- Manipulator Arm -->
+  <xacro:property name="arm_x" value="0.08" />
+  <xacro:property name="arm_z" value="0.015" />
+  <xacro:property name="al1" value="0.04" />
+  <xacro:property name="al2" value="0.10" />
+  <xacro:property name="al3" value="0.10" />
+  <!-- Arm Base -->
+  <joint name="arm_base_joint" type="revolute">
+    <parent link="base_link"/><child link="arm_base_link"/>
+    <origin xyz="${arm_x} 0 ${arm_z}" rpy="0 0 0"/>
+    <axis xyz="0 0 1"/><limit lower="-3.14" upper="3.14" effort="5" velocity="1.0"/>
+  </joint>
+  <link name="arm_base_link">
+    <visual><geometry><cylinder radius="0.03" length="${al1}"/></geometry><material name="green"/></visual>
+    <xacro:box_inertia m="0.1" x="0.03" y="0.03" z="${al1}"/>
+  </link>
+  <!-- Arm Link 1 -->
+  <joint name="arm_joint_1" type="revolute">
+    <parent link="arm_base_link"/><child link="arm_link_1"/>
+    <origin xyz="0 0 ${al1/2}" rpy="0 0 0"/>
+    <axis xyz="0 1 0"/><limit lower="-1.57" upper="1.57" effort="5" velocity="1.0"/>
+  </joint>
+  <link name="arm_link_1">
+    <visual><origin xyz="0 0 ${al2/2}"/><geometry><box size="0.02 0.02 ${al2}"/></geometry><material name="dark_gray"/></visual>
+    <xacro:box_inertia m="0.1" x="0.02" y="0.02" z="${al2}"/>
+  </link>
+  <!-- Arm Link 2 -->
+  <joint name="arm_joint_2" type="revolute">
+    <parent link="arm_link_1"/><child link="arm_link_2"/>
+    <origin xyz="0 0 ${al2}" rpy="0 0 0"/>
+    <axis xyz="0 1 0"/><limit lower="-2.5" upper="2.5" effort="5" velocity="1.0"/>
+  </joint>
+  <link name="arm_link_2">
+    <visual><origin xyz="0 0 ${al3/2}"/><geometry><box size="0.015 0.015 ${al3}"/></geometry><material name="green"/></visual>
+    <xacro:box_inertia m="0.05" x="0.015" y="0.015" z="${al3}"/>
+  </link>
 </robot>
